File: Whisker-LogicProbe/Whiskers-LogicProbe.sch (KiCad schematic (older format))
At the start: 34 parts, among them J1 Conn_01x10_Male, J10 Conn_01x04_Male, J11 Conn_01x04_Male, J9 USB_B_Micro, U1 SN65LVDS(T)348, U2 MIC5504-3.3YM5

Commit message: Updated to use the proper LVDS receiver chip (560Mb/s one)
Parts:
- removed R10, R9: 250, Resistor_SMD:R_0603_1608Metric, symbol Device:R_Small
- removed U1: SN65LVDS(T)348, Package_SO:TSSOP-16_4.4x5mm_P0.65mm, symbol WhiskersLib:SN65LVDS(T)348
- added C7, C8, C9: 0.1uF, Capacitor_SMD:C_0603_1608Metric, symbol Device:C_Small
- added FID1, FID2, FID3: Fiducial, Fiducial:Fiducial_0.5mm_Mask1mm, symbol Mechanical:Fiducial
- added H1, H2: MountingHole_Pad, MountingHole:MountingHole_3.2mm_M3_DIN965_Pad, symbol Mechanical:MountingHole_Pad
- added U1: SN65LVDS(T)352, Package_SO:TSSOP-24_4.4x7.8mm_P0.65mm, symbol WhiskersLib:SN65LVDS(T)352
Connections:
- wire segments 145 -> 170
Other:
- moved on the sheet: C3, C4, C5, C6, J1, J10, J11, R1, R11, R12, R13, R14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
